File: Electrical files/Wiring diagram/Wiring diagram.kicad_sch (KiCad schematic)
At the start: 0 parts

Commit message: wiring diagram
Parts:
- added J1: RS PRO 811-7216 C14, symbol New_Library:IEC_C14_Inlet_Fuse_DPST_RS_811-7216
- added LC1, LC2, LC3, LC4: Phidgets 3135_0 50kg, symbol New_Library:LoadCell_Phidgets_3135_0_50kg
- added PS1: RS PRO 262-9109 5V 18A, symbol New_Library:RSPRO_262-9109_5V_90W
- added PS2: MEAN WELL HRP-300-24, symbol New_Library:HRP-300-24
- added U1: ESP32-DEV-38P, symbol ESP32-DEV-38P:ESP32-DEV-38P
- added U2, U6, U7, U8: Adafruit 4538 NAU7802, symbol New_Library:NAU7802_ADC_Adafruit_4538
- added U4: Adafruit 2019 MMA8451 IMU, symbol New_Library:MMA8451_Accel_Adafruit_2019
- added U5: SparkFun 16784 Qwiic Mux 8ch, symbol New_Library:Qwiic_Mux_TCA9548A_SparkFun_16784
Connections:
- new net: PS1.6 (+V), U2.1 (VIN), U6.1 (VIN), U7.1 (VIN), U8.1 (VIN)
- new net: U5.14 (SC2), U7.4 (SCL)
- new net: U5.13 (SD2), U7.5 (SDA)
- new net: LC3.1 (E+_(red)), U7.6 (E+)
- new net: LC3.2 (E-_(black)), U7.7 (E-)
- new net: LC3.3 (S+_(green)), U7.8 (A+)
- new net: LC3.4 (S-_(white)), U7.9 (A-)
- new net: J1.3 (L_OUT), PS1.1 (AC/L), PS2.1 (AC/L)
- new net: J1.4 (N_OUT), PS1.2 (AC/N), PS2.2 (AC/N)
- new net: LC4.1 (E+_(red)), U8.6 (E+)
- new net: LC4.2 (E-_(black)), U8.7 (E-)
- new net: LC4.3 (S+_(green)), U8.8 (A+)
- new net: LC4.4 (S-_(white)), U8.9 (A-)
- new net: LC2.1 (E+_(red)), U2.6 (E+)
- new net: LC2.2 (E-_(black)), U2.7 (E-)
- new net: LC2.3 (S+_(green)), U2.8 (A+)
- new net: LC2.4 (S-_(white)), U2.9 (A-)
- new net: U5.10 (SC0), U6.4 (SCL)
- new net: U5.9 (SD0), U6.5 (SDA)
- new net: LC1.1 (E+_(red)), U6.6 (E+)
- new net: LC1.2 (E-_(black)), U6.7 (E-)
- new net: LC1.3 (S+_(green)), U6.8 (A+)
- new net: LC1.4 (S-_(white)), U6.9 (A-)
- new net: U5.16 (SC3), U8.4 (SCL)
- new net: U5.15 (SD3), U8.5 (SDA)
- new net: U1.1 (3V3), U5.1 (3V3)
- new net: U2.4 (SCL), U5.12 (SC1)
- new net: U2.5 (SDA), U5.11 (SD1)
- new net GND: U1.20 (GND), U2.3 (GND), U4.3 (GND), U5.2 (GND), U6.3 (GND), U7.3 (GND), U8.3 (GND)
Other:
- added sheet Loadcell (untitled.kicad_sch)
- added sheet Power delivery (untitled.kicad_sch)
- note added: "Not sure if esp32 can give the required current"

Commit message: First iteration of wiring diagram
Parts:
- added M1, M2: Linear actuator + encoder, symbol Pivot:LinearActuator_Encoder_6pin
- added U3: DFRobot DFR0601 2ch 12A, symbol Pivot:MotorDriver_DFRobot_DFR0601
Connections:
- net GND: now also U1.30 (GPIO17), U5.6 (ADR0), U5.7 (ADR1), U5.8 (ADR2), M1.4 (ENC-), M2.4 (ENC-), U3.10 (GND), U3.5 (GND), U3.9 (INB2)
- net at PS1.6 (+V), U2.1 (VIN), U6.1 (VIN)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: now also M1.3 (ENC+), M2.3 (ENC+), U3.1 (VCC), U3.6 (VCC)
- net at J1.5 (PE): now also PS1.3 (FG), PS2.3 (FG)
- net at PS2.4 (-V): now also U3.15 (P-)
- net at PS2.6 (+V): now also U3.16 (P+)
- net at U1.10 (GPIO26): now also U3.7 (PWM2)
- net at U1.27 (GPIO19): now also U3.3 (INA1)
- net at U1.28 (GPIO18): now also U3.4 (INB1)
- net at U1.29 (GPIO5): now also U3.8 (INA2)
- net at U1.36 (SD1_/_GPIO8): now also U5.3 (SDA)
- net at U1.37 (SD0_/_GPIO7): now also U5.4 (SCL)
- net at U1.5 (GPIO34): now also M1.5 (ENC_A)
- net at U1.6 (GPIO35): now also M1.6 (ENC_B)
- net at U1.7 (GPIO32): now also M2.5 (ENC_A)
- net at U1.8 (GPIO33): now also M2.6 (ENC_B)
- net at U1.9 (GPIO25): now also U3.2 (PWM1)
- new net: M2.1 (MOTOR+), U3.13 (M2_A)
- new net: M2.2 (MOTOR-), U3.14 (M2_B)
- new net: M1.1 (MOTOR+), U3.11 (M1_A)
- new net: M1.2 (MOTOR-), U3.12 (M1_B)
Other:
- added sheet Motordriver and actuators (untitled.kicad_sch)
- moved on the sheet: U1, U4, U5
